Commit message: Increate wheel weight to prevent body drift due to stepping cmd_vel

File: urdf/wheel/vwheel.urdf.xacro (robot description, xacro)
@@ -6,5 +6,5 @@
   <xacro:property name="wheel_inertial_length" value="0.03"/>
   <xacro:property name="wheel_collition_length" value="0.001"/>
-  <xacro:property name="wheel_mass" value="0.823"/>
+  <xacro:property name="wheel_mass" value="2.5"/>
   <xacro:macro name="wheel_v0" params="prefix parent *joint_origin *joint_axis">
     <joint name="${prefix}_wheel_joint" type="continuous">

Commit message: revert wheel_length

File: urdf/wheel/vwheel.urdf.xacro (robot description, xacro)
@@ -4,7 +4,6 @@
   <xacro:include filename="$(find megarover_samples_ros2)/urdf/wheel/wheel.gazebo.xacro"/>
   <xacro:property name="wheel_radius" value="0.076"/>
-  <xacro:property name="wheel_inertial_length" value="0.03"/>
-  <xacro:property name="wheel_collition_length" value="0.001"/>
-  <xacro:property name="wheel_mass" value="2.5"/>
+  <xacro:property name="wheel_length" value="0.03"/>
+  <xacro:property name="wheel_mass" value="0.823"/>
   <xacro:macro name="wheel_v0" params="prefix parent *joint_origin *joint_axis">
     <joint name="${prefix}_wheel_joint" type="continuous">
@@ -23,5 +22,5 @@
         <origin xyz="0 0 0" rpy="${-M_PI/2} 0 0"/>
         <geometry>
-          <cylinder radius="${wheel_radius}" length="${wheel_collition_length}"/>
+          <cylinder radius="${wheel_radius}" length="${wheel_length}"/>
         </geometry>
       </collision>
@@ -29,5 +28,5 @@
         <origin xyz="0 0 0" rpy="${-M_PI/2} 0 0"/>
         <xacro:cylinder_inertial mass="${wheel_mass}"
-          radius="${wheel_radius}" length="${wheel_inertial_length}"/>
+          radius="${wheel_radius}" length="${wheel_length}"/>
       </inertial>
     </link>

Commit message: fixed left wheel visual

File: urdf/wheel/vwheel.urdf.xacro (robot description, xacro)
@@ -18,6 +18,6 @@
           <origin xyz="0 0 0" rpy="${M_PI/2} 0 0"/>
         </xacro:if>
-        <xacro:if value="${prefix=='right'}">
-          <origin xyz="0 0 0" rpy="${M_PI/2} 0 0"/>
+        <xacro:if value="${prefix=='left'}">
+          <origin xyz="0 0 0" rpy="-${M_PI/2} 0 0"/>
         </xacro:if>
         <geometry>
