Commit message: spawn from xacro , remove unused sdf

File: urdf/lrf/lrf.gazebo.xacro (robot description, xacro)
@@ -27,8 +27,10 @@
           </noise>
         </ray>
-        <plugin name="gazebo_ros_${prefix}_lrf_controller" filename="libgazebo_ros_laser.so">
-          <!-- <topicName>${prefix}/scan</topicName> -->
-          <topicName>/scan</topicName>
-          <frameName>${prefix}_lrf_link</frameName>
+        <plugin name='gazebo_ros_front_lrf_controller' filename='libgazebo_ros_ray_sensor.so'>
+          <ros>
+            <remapping>~/out:=scan</remapping>
+          </ros>
+          <output_type>sensor_msgs/LaserScan</output_type>
+          <!-- <frame_name> ommited, will default to ${prefix}_lrf_link-->
         </plugin>
       </sensor>

File: urdf/wheel/wheel.transmission.xacro (robot description, xacro)
@@ -2,14 +2,6 @@
 <robot xmlns:xacro="http://ros.org/wiki/xacro">
   <xacro:macro name="wheel_trans_v0" params="prefix">
-    <transmission name="${prefix}_wheel_trans">
-      <type>transmission_interface/SimpleTransmission</type>
-      <joint name="${prefix}_wheel_joint">
-        <hardwareInterface>hardware_interface/VelocityJointInterface</hardwareInterface>
-      </joint>
-      <actuator name="${prefix}_wheel_motor">
-        <hardwareInterface>hardware_interface/VelocityJointInterface</hardwareInterface>
-        <mechanicalReduction>30</mechanicalReduction>
-      </actuator>
-    </transmission>
+    <!-- <transmission> ommited in ros2-->
+    <!-- todo ros2_control system -->
   </xacro:macro>
 </robot>
