Commit message: fixed URDF

File: urdf/camera/camera.urdf.xacro (robot description, xacro)
@@ -13,5 +13,5 @@
         <origin xyz="0 0 0" rpy="0 0 0"/>
         <geometry>
-	      <box size="0.02 0.097 0.02"/>
+          <box size="0.02 0.097 0.02"/>
         </geometry>
       </visual>
@@ -19,5 +19,5 @@
         <origin xyz="0 0 0" rpy="0 0 0"/>
         <geometry>
-	      <box size="0.02 0.097 0.02"/>
+          <box size="0.02 0.097 0.02"/>
         </geometry>
       </collision>
