Commit message: changed position and spec of lrf

File: robots/vmegarover.urdf.xacro (robot description, xacro)
@@ -22,11 +22,11 @@
   </xacro:wheel_v0>
   <!-- Front LRF -->
+  <!-- <xacro:lrf_v0 prefix="front" parent="base_link">
+    <origin xyz="0.099 0 0.1015"/>
+  </xacro:lrf_v0> -->
+  <!-- Front LRF Upper-->
   <xacro:lrf_v0 prefix="front" parent="base_link">
-    <origin xyz="0.099 0 0.1015"/>
+    <origin xyz="0.099 0 0.2155"  rpy="${M_PI} 0 0" />
   </xacro:lrf_v0>
-  <!-- Front LRF Upper-->
-  <!-- <xacro:lrf_v0 prefix="front" parent="base_link">
-    <origin xyz="0.099 0 0.2155"  rpy="${M_PI} 0 0" />
-  </xacro:lrf_v0> -->
   <!-- Rear LRF -->
   <!-- xacro:lrf_v0 prefix="rear" parent="base_link">
@@ -55,8 +55,8 @@
   <!-- LRF -->
   <xacro:lrf_gazebo_v0 prefix="front"
-                       min_rad="-1.57" max_rad="1.57"
-                       min_range="0.06" max_range="4.0"/>
+                       min_rad="-${M_PI}" max_rad="${M_PI}"
+                       min_range="0.06" max_range="10.0"/>
   <!-- xacro:lrf_gazebo_v0 prefix="rear"
                        min_rad="-1.57" max_rad="1.57"
-                       min_range="0.06" max_range="4.0"/ -->
+                       min_range="0.06" max_range="10.0"/ -->
 </robot>

Commit message: WIP: support of ros2_control , TODO: fix odometry

File: robots/vmegarover.urdf.xacro (robot description, xacro)
@@ -1,4 +1,5 @@
 <?xml version="1.0"?>
 <robot name="vmegarover" xmlns:xacro="http://ros.org/wiki/xacro">
+  <xacro:arg name="use_ros2_control" default="false" />
   <xacro:include filename="$(find megarover_samples_ros2)/urdf/body/vbody.urdf.xacro"/>
   <xacro:include filename="$(find megarover_samples_ros2)/urdf/wheel/vwheel.urdf.xacro"/>
@@ -39,24 +40,53 @@
     <origin xyz="0.099 0 0.1015"/>
   </joint>
-  <!-- ===============  Transmission =============== -->
-  <xacro:wheel_trans_v0 prefix="right"/>
-  <xacro:wheel_trans_v0 prefix="left"/>
   <!-- =============== Gazebo =============== -->
-  <gazebo>
-    <plugin name='diff_drive' filename='libgazebo_ros_diff_drive.so'>
-      <ros>
-        <namespace>/vmegarover</namespace>
-      </ros>
-      <update_rate>50</update_rate>
-      <left_joint>left_wheel_joint</left_joint>
-      <right_joint>right_wheel_joint</right_joint>
-      <wheel_separation>0.284</wheel_separation>
-      <wheel_diameter>0.152</wheel_diameter>
-      <publish_odom>true</publish_odom>
-      <publish_odom_tf>true</publish_odom_tf>
-      <odometry_frame>odom</odometry_frame>
-      <robot_base_frame>base_footprint</robot_base_frame>
-    </plugin>
-  </gazebo>
+  <xacro:if value="$(arg use_ros2_control)">
+    <!-- use ros2_control -->
+    <ros2_control name="GazeboSystem" type="system">
+      <hardware>
+        <plugin>gazebo_ros2_control/GazeboSystem</plugin>
+      </hardware>
+      <joint name="left_wheel_joint">
+        <command_interface name="velocity">
+          <param name="min">-1</param>
+          <param name="max">1</param>
+        </command_interface>
+        <state_interface name="position"/>
+        <state_interface name="velocity"/>
+      </joint>
+      <joint name="right_wheel_joint">
+        <command_interface name="velocity">
+          <param name="min">-1</param>
+          <param name="max">1</param>
+        </command_interface>
+        <state_interface name="position"/>
+        <state_interface name="velocity"/>
+      </joint>
+    </ros2_control>
+    <gazebo>
+      <plugin name="gazebo_ros2_control" filename="libgazebo_ros2_control.so">
+        <parameters>$(find megarover_samples_ros2)/config/diff_drive_controller.yaml</parameters>
+      </plugin>
+    </gazebo>
+  </xacro:if>
+  <xacro:unless value="$(arg use_ros2_control)">
+    <!-- use libgazebo_ros_diff_drive.so -->
+    <gazebo>
+      <plugin name='diff_drive_controller' filename='libgazebo_ros_diff_drive.so'>
+        <ros>
+          <namespace>/vmegarover</namespace>
+        </ros>
+        <update_rate>50</update_rate>
+        <left_joint>left_wheel_joint</left_joint>
+        <right_joint>right_wheel_joint</right_joint>
+        <wheel_separation>0.284</wheel_separation>
+        <wheel_diameter>0.152</wheel_diameter>
+        <publish_odom>true</publish_odom>
+        <publish_odom_tf>true</publish_odom_tf>
+        <odometry_frame>odom</odometry_frame>
+        <robot_base_frame>base_footprint</robot_base_frame>
+      </plugin>
+    </gazebo>
+  </xacro:unless>
   <!-- Base -->
   <xacro:base_gazebo_v0/>

File: urdf/wheel/vwheel.urdf.xacro (robot description, xacro)
@@ -2,5 +2,4 @@
 <robot xmlns:xacro="http://ros.org/wiki/xacro">
   <xacro:include filename="$(find megarover_samples_ros2)/urdf/common.xacro"/>
-  <xacro:include filename="$(find megarover_samples_ros2)/urdf/wheel/wheel.transmission.xacro"/>
   <xacro:include filename="$(find megarover_samples_ros2)/urdf/wheel/wheel.gazebo.xacro"/>
   <xacro:property name="wheel_radius" value="0.076"/>

Commit message: WIP: migration to ignition gazebo from classic

File: robots/vmegarover.urdf.xacro (robot description, xacro)
@@ -1,4 +1,5 @@
 <?xml version="1.0"?>
 <robot name="vmegarover" xmlns:xacro="http://ros.org/wiki/xacro">
+  <xacro:arg name="gazebo" default="classic" />
   <xacro:arg name="use_ros2_control" default="false" />
   <xacro:include filename="$(find megarover_samples_ros2)/urdf/body/vbody.urdf.xacro"/>
@@ -58,52 +59,104 @@
   </joint>
   <!-- =============== Gazebo =============== -->
-  <xacro:if value="$(arg use_ros2_control)">
-    <!-- use ros2_control -->
-    <ros2_control name="GazeboSystem" type="system">
-      <hardware>
-        <plugin>gazebo_ros2_control/GazeboSystem</plugin>
-      </hardware>
-      <joint name="left_wheel_joint">
-        <command_interface name="velocity">
-          <param name="min">-1</param>
-          <param name="max">1</param>
-        </command_interface>
-        <state_interface name="position"/>
-        <state_interface name="velocity"/>
-      </joint>
-      <joint name="right_wheel_joint">
-        <command_interface name="velocity">
-          <param name="min">-1</param>
-          <param name="max">1</param>
-        </command_interface>
-        <state_interface name="position"/>
-        <state_interface name="velocity"/>
-      </joint>
-    </ros2_control>
-    <gazebo>
-      <plugin name="gazebo_ros2_control" filename="libgazebo_ros2_control.so">
-        <parameters>$(find megarover_samples_ros2)/config/diff_drive_controller.yaml</parameters>
-      </plugin>
-    </gazebo>
+  <xacro:if value="${'$(arg gazebo)' == 'classic'}">
+    <xacro:if value="$(arg use_ros2_control)">
+      <!-- use ros2_control -->
+      <ros2_control name="GazeboSystem" type="system">
+        <hardware>
+          <plugin>gazebo_ros2_control/GazeboSystem</plugin>
+        </hardware>
+        <joint name="left_wheel_joint">
+          <command_interface name="velocity">
+            <param name="min">-1</param>
+            <param name="max">1</param>
+          </command_interface>
+          <state_interface name="position"/>
+          <state_interface name="velocity"/>
+        </joint>
+        <joint name="right_wheel_joint">
+          <command_interface name="velocity">
+            <param name="min">-1</param>
+            <param name="max">1</param>
+          </command_interface>
+          <state_interface name="position"/>
+          <state_interface name="velocity"/>
+        </joint>
+      </ros2_control>
+      <gazebo>
+        <plugin name="gazebo_ros2_control" filename="libgazebo_ros2_control.so">
+          <parameters>$(find megarover_samples_ros2)/config/diff_drive_controller.yaml</parameters>
+        </plugin>
+      </gazebo>
+    </xacro:if>
+    <xacro:unless value="$(arg use_ros2_control)">
+      <!-- use libgazebo_ros_diff_drive.so -->
+      <gazebo>
+        <plugin name='diff_drive_controller' filename='libgazebo_ros_diff_drive.so'>
+          <ros>
+            <namespace>/vmegarover</namespace>
+          </ros>
+          <update_rate>50</update_rate>
+          <left_joint>left_wheel_joint</left_joint>
+          <right_joint>right_wheel_joint</right_joint>
+          <wheel_separation>0.284</wheel_separation>
+          <wheel_diameter>0.152</wheel_diameter>
+          <publish_odom>true</publish_odom>
+          <publish_odom_tf>true</publish_odom_tf>
+          <odometry_frame>odom</odometry_frame>
+          <robot_base_frame>base_footprint</robot_base_frame>
+        </plugin>
+      </gazebo>
+    </xacro:unless>
   </xacro:if>
-  <xacro:unless value="$(arg use_ros2_control)">
-    <!-- use libgazebo_ros_diff_drive.so -->
-    <gazebo>
-      <plugin name='diff_drive_controller' filename='libgazebo_ros_diff_drive.so'>
-        <ros>
-          <namespace>/vmegarover</namespace>
-        </ros>
-        <update_rate>50</update_rate>
-        <left_joint>left_wheel_joint</left_joint>
-        <right_joint>right_wheel_joint</right_joint>
-        <wheel_separation>0.284</wheel_separation>
-        <wheel_diameter>0.152</wheel_diameter>
-        <publish_odom>true</publish_odom>
-        <publish_odom_tf>true</publish_odom_tf>
-        <odometry_frame>odom</odometry_frame>
-        <robot_base_frame>base_footprint</robot_base_frame>
-      </plugin>
-    </gazebo>
-  </xacro:unless>
+  <xacro:if value="${'$(arg gazebo)' == 'ignition'}">
+    <xacro:if value="$(arg use_ros2_control)">
+      <!-- use ros2_control -->
+      <ros2_control name="GazeboSystem" type="system">
+        <hardware>
+          <plugin>gz_ros2_control/GazeboSimSystem</plugin>
+        </hardware>
+        <joint name="left_wheel_joint">
+          <command_interface name="velocity">
+            <param name="min">-1</param>
+            <param name="max">1</param>
+          </command_interface>
+          <state_interface name="position"/>
+          <state_interface name="velocity"/>
+        </joint>
+        <joint name="right_wheel_joint">
+          <command_interface name="velocity">
+            <param name="min">-1</param>
+            <param name="max">1</param>
+          </command_interface>
+          <state_interface name="position"/>
+          <state_interface name="velocity"/>
+        </joint>
+      </ros2_control>
+      <gazebo>
+        <plugin name="gz_ros2_control::GazeboSimROS2ControlPlugin" filename="gz_ros2_control-system">
+          <parameters>$(find megarover_samples_ros2)/config/diff_drive_controller.yaml</parameters>
+        </plugin>
+      </gazebo>
+    </xacro:if>
+    <xacro:unless value="$(arg use_ros2_control)">
+      <!-- use ignition-gazebo-diff-drive-system -->
+      <gazebo>
+        <plugin name='ignition::gazebo::systems::DiffDrive' filename='ignition-gazebo-diff-drive-system'>
+          <ros>
+            <namespace>/vmegarover</namespace>
+          </ros>
+          <update_rate>50</update_rate>
+          <left_joint>left_wheel_joint</left_joint>
+          <right_joint>right_wheel_joint</right_joint>
+          <wheel_separation>0.284</wheel_separation>
+          <wheel_diameter>0.152</wheel_diameter>
+          <publish_odom>true</publish_odom>
+          <publish_odom_tf>true</publish_odom_tf>
+          <odometry_frame>odom</odometry_frame>
+          <robot_base_frame>base_footprint</robot_base_frame>
+        </plugin>
+      </gazebo>
+    </xacro:unless>
+  </xacro:if>
   <!-- Base -->
   <xacro:base_gazebo_v0/>
@@ -112,5 +165,6 @@
   <xacro:wheel_gazebo_v0 prefix="left"/>
   <!-- LRF -->
-  <xacro:lrf_gazebo_v0 prefix="front"
+  <xacro:lrf_gazebo_v0 gazebo="$(arg gazebo)"
+                       prefix="front"
                        min_rad="-3.14" max_rad="3.14"
                        min_range="0.06" max_range="10.0"/>
@@ -119,4 +173,11 @@
                        min_range="0.06" max_range="10.0"/ -->
   <!-- Camera -->
-  <xacro:camera_gazebo_v0 prefix="front"/>
+  <xacro:camera_gazebo_v0 gazebo="$(arg gazebo)" prefix="front"/>
+  <xacro:if value="${'$(arg gazebo)' == 'ignition'}">
+    <gazebo>
+      <plugin filename="ignition-gazebo-sensors-system" name="ignition::gazebo::systems::Sensors">
+        <render_engine>ogre2</render_engine>
+      </plugin>
+    </gazebo>
+  </xacro:if>
 </robot>

File: urdf/camera/camera.gazebo.xacro (robot description, xacro)
@@ -1,38 +1,63 @@
 <?xml version="1.0"?>
 <robot xmlns:xacro="http://ros.org/wiki/xacro">
-  <xacro:macro name="camera_gazebo_v0" params="prefix">
+  <xacro:macro name="camera_gazebo_v0" params="gazebo prefix">
     <gazebo reference="${prefix}_camera_link">
-      <sensor name="${prefix}_camera_sensor" type="depth">
-        <pose>0 0 0 0 0 0</pose>
-        <update_rate>30.0</update_rate>
-        <camera name="camera">
-          <horizontal_fov>1.56207</horizontal_fov>
-          <image>
-            <width>640</width>
-            <height>400</height>
-            <format>R8G8B8</format>
-          </image>
-          <clip>
-            <near>0.02</near>
-            <far>8.0</far>
-          </clip>
-          <noise>
-            <type>gaussian</type>
-            <mean>0.0</mean>
-            <stddev>0.007</stddev>
-          </noise>
-        </camera>
-        <plugin name="camera_controller" filename="libgazebo_ros_camera.so">
-          <min_depth>0.2</min_depth>
-          <max_depth>8.0</max_depth>
-          <hack_baseline>0.07</hack_baseline>
-          <frame_name>camera_depth_link</frame_name>
-          <distortion_k1>0.0</distortion_k1>
-          <distortion_k2>0.0</distortion_k2>
-          <distortion_k3>0.0</distortion_k3>
-          <distortion_t1>0.0</distortion_t1>
-          <distortion_t2>0.0</distortion_t2>
-        </plugin>
-      </sensor>
+      <xacro:if value="${gazebo == 'classic'}">
+        <sensor name="${prefix}_camera_sensor" type="depth">
+          <pose>0 0 0 0 0 0</pose>
+          <update_rate>30.0</update_rate>
+          <camera name="camera">
+            <horizontal_fov>1.56207</horizontal_fov>
+            <image>
+              <width>640</width>
+              <height>400</height>
+              <format>R8G8B8</format>
+            </image>
+            <clip>
+              <near>0.02</near>
+              <far>8.0</far>
+            </clip>
+            <noise>
+              <type>gaussian</type>
+              <mean>0.0</mean>
+              <stddev>0.007</stddev>
+            </noise>
+          </camera>
+          <plugin name="camera_controller" filename="libgazebo_ros_camera.so">
+            <min_depth>0.2</min_depth>
+            <max_depth>8.0</max_depth>
+            <hack_baseline>0.07</hack_baseline>
+            <frame_name>camera_depth_link</frame_name>
+            <distortion_k1>0.0</distortion_k1>
+            <distortion_k2>0.0</distortion_k2>
+            <distortion_k3>0.0</distortion_k3>
+            <distortion_t1>0.0</distortion_t1>
+            <distortion_t2>0.0</distortion_t2>
+          </plugin>
+        </sensor>
+      </xacro:if>
+      <xacro:if value="${gazebo == 'ignition'}">
+        <sensor name="${prefix}_camera_sensor" type="depth_camera">
+          <pose>0 0 0 0 0 0</pose>
+          <update_rate>30.0</update_rate>
+          <camera>
+            <horizontal_fov>1.56207</horizontal_fov>
+            <image>
+              <width>640</width>
+              <height>400</height>
+              <format>R8G8B8</format>
+            </image>
+            <clip>
+              <near>0.02</near>
+              <far>8.0</far>
+            </clip>
+            <noise>
+              <type>gaussian</type>
+              <mean>0.0</mean>
+              <stddev>0.007</stddev>
+            </noise>
+          </camera>
+        </sensor>
+      </xacro:if>
     </gazebo>
   </xacro:macro>

File: urdf/lrf/lrf.gazebo.xacro (robot description, xacro)
@@ -1,39 +1,68 @@
 <?xml version="1.0"?>
 <robot xmlns:xacro="http://ros.org/wiki/xacro">
-  <xacro:macro name="lrf_gazebo_v0" params="prefix min_rad max_rad min_range max_range">
+  <xacro:macro name="lrf_gazebo_v0" params="gazebo prefix min_rad max_rad min_range max_range">
     <gazebo reference="${prefix}_lrf_link">
-      <sensor type="ray" name="${prefix}_lrf_sensor">
-        <pose>0 0 0 0 0 0</pose>
-        <visualize>false</visualize>
-        <update_rate>40</update_rate>
-        <ray>
-          <scan>
-            <horizontal>
-              <samples>1000</samples>
-              <resolution>1</resolution>
-              <min_angle>${min_rad}</min_angle>
-              <max_angle>${max_rad}</max_angle>
-            </horizontal>
-          </scan>
-          <range>
-            <min>${min_range}</min>
-            <max>${max_range}</max>
-            <resolution>0.001</resolution>
-          </range>
-          <noise>
-            <type>gaussian</type>
-            <mean>0.0</mean>
-            <stddev>0.03</stddev>
-          </noise>
-        </ray>
-        <plugin name='gazebo_ros_front_lrf_controller' filename='libgazebo_ros_ray_sensor.so'>
-          <ros>
-            <remapping>~/out:=scan</remapping>
-          </ros>
-          <output_type>sensor_msgs/LaserScan</output_type>
-          <!-- <frame_name> ommited, will default to ${prefix}_lrf_link-->
-          <frame_name>${prefix}_lrf_link</frame_name>
-        </plugin>
-      </sensor>
+      <xacro:if value="${gazebo == 'classic'}">
+        <sensor type="ray" name="${prefix}_lrf_sensor">
+          <pose>0 0 0 0 0 0</pose>
+          <visualize>false</visualize>
+          <update_rate>40</update_rate>
+          <ray>
+            <scan>
+              <horizontal>
+                <samples>1000</samples>
+                <resolution>1</resolution>
+                <min_angle>${min_rad}</min_angle>
+                <max_angle>${max_rad}</max_angle>
+              </horizontal>
+            </scan>
+            <range>
+              <min>${min_range}</min>
+              <max>${max_range}</max>
+              <resolution>0.001</resolution>
+            </range>
+            <noise>
+              <type>gaussian</type>
+              <mean>0.0</mean>
+              <stddev>0.03</stddev>
+            </noise>
+          </ray>
+          <plugin name='gazebo_ros_front_lrf_controller' filename='libgazebo_ros_ray_sensor.so'>
+            <ros>
+              <remapping>~/out:=scan</remapping>
+            </ros>
+            <output_type>sensor_msgs/LaserScan</output_type>
+            <!-- <frame_name> ommited, will default to ${prefix}_lrf_link-->
+            <frame_name>${prefix}_lrf_link</frame_name>
+          </plugin>
+        </sensor>
+      </xacro:if>
+      <xacro:if value="${gazebo == 'ignition'}">
+        <sensor type="gpu_lidar" name="${prefix}_lrf_sensor">
+          <pose>0 0 0 0 0 0</pose>
+          <visualize>false</visualize>
+          <update_rate>40</update_rate>
+          <lidar>
+            <scan>
+              <horizontal>
+                <samples>1000</samples>
+                <resolution>1</resolution>
+                <min_angle>${min_rad}</min_angle>
+                <max_angle>${max_rad}</max_angle>
+              </horizontal>
+            </scan>
+            <range>
+              <min>${min_range}</min>
+              <max>${max_range}</max>
+              <resolution>0.001</resolution>
+            </range>
+            <noise>
+              <type>gaussian</type>
+              <mean>0.0</mean>
+              <stddev>0.03</stddev>
+            </noise>
+          </lidar>
+        </sensor>
+      </xacro:if>
     </gazebo>
   </xacro:macro>

Commit message: fix: fixed model path format, remove topic_relay

File: robots/vmegarover.urdf.xacro (robot description, xacro)
@@ -85,4 +85,8 @@
       <gazebo>
         <plugin name="gazebo_ros2_control" filename="libgazebo_ros2_control.so">
+          <ros>
+            <remapping>~/cmd_vel_unstamped:=/cmd_vel</remapping>
+            <remapping>~/odom:=/odom</remapping>
+          </ros>
           <parameters>$(find megarover_samples_ros2)/config/diff_drive_controller.yaml</parameters>
         </plugin>
@@ -94,5 +98,5 @@
         <plugin name='diff_drive_controller' filename='libgazebo_ros_diff_drive.so'>
           <ros>
-            <namespace>/vmegarover</namespace>
+            <namespace>/</namespace>
           </ros>
           <update_rate>50</update_rate>

File: urdf/body/vbody.urdf.xacro (robot description, xacro)
@@ -11,10 +11,10 @@
       <visual>
         <geometry>
-          <mesh filename="package://megarover_samples_ros2/models/vmegarover/meshes/dae/vmega_body.dae"/>
+          <mesh filename="file://$(find megarover_samples_ros2)/models/vmegarover/meshes/dae/vmega_body.dae"/>
         </geometry>
       </visual>
       <collision>
         <geometry>
-          <mesh filename="package://megarover_samples_ros2/models/vmegarover/meshes/stl/vmega_body.stl"/>
+          <mesh filename="file://$(find megarover_samples_ros2)/models/vmegarover/meshes/stl/vmega_body.stl"/>
         </geometry>
       </collision>

File: urdf/lrf/lrf.urdf.xacro (robot description, xacro)
@@ -12,10 +12,10 @@
       <visual>
         <geometry>
-          <mesh filename="package://megarover_samples_ros2/models/vmegarover/meshes/dae/lrf.dae"/>
+          <mesh filename="file://$(find megarover_samples_ros2)/models/vmegarover/meshes/dae/lrf.dae"/>
         </geometry>
       </visual>
       <collision>
         <geometry>
-          <mesh filename="package://megarover_samples_ros2/models/vmegarover/meshes/stl/lrf.stl"/>
+          <mesh filename="file://$(find megarover_samples_ros2)/models/vmegarover/meshes/stl/lrf.stl"/>
         </geometry>
       </collision>

File: urdf/wheel/vwheel.urdf.xacro (robot description, xacro)
@@ -16,5 +16,5 @@
       <visual>
         <geometry>
-          <mesh filename="package://megarover_samples_ros2/models/vmegarover/meshes/dae/vmega_wheel.dae"/>
+          <mesh filename="file://$(find megarover_samples_ros2)/models/vmegarover/meshes/dae/vmega_wheel.dae"/>
         </geometry>
       </visual>
