Commit message: removed code for Gazebo Classic

File: robots/vmegarover.urdf.xacro (robot description, xacro)
@@ -1,5 +1,5 @@
 <?xml version="1.0"?>
 <robot name="vmegarover" xmlns:xacro="http://ros.org/wiki/xacro">
-  <xacro:arg name="gazebo" default="classic" />
+  <xacro:arg name="gazebo" default="ignition" />
   <xacro:arg name="use_ros2_control" default="false" />
   <xacro:include filename="$(find megarover_samples_ros2)/urdf/body/vbody.urdf.xacro"/>
@@ -58,63 +58,4 @@
     <child link="camera_depth_link"/>
   </joint>
-  <!-- =============== Gazebo =============== -->
-  <xacro:if value="${'$(arg gazebo)' == 'classic'}">
-    <xacro:if value="$(arg use_ros2_control)">
-      <!-- use ros2_control -->
-      <ros2_control name="GazeboSystem" type="system">
-        <hardware>
-          <plugin>gazebo_ros2_control/GazeboSystem</plugin>
-        </hardware>
-        <joint name="left_wheel_joint">
-          <command_interface name="velocity">
-            <param name="min">-1</param>
-            <param name="max">1</param>
-          </command_interface>
-          <state_interface name="position"/>
-          <state_interface name="velocity"/>
-        </joint>
-        <joint name="right_wheel_joint">
-          <command_interface name="velocity">
-            <param name="min">-1</param>
-            <param name="max">1</param>
-          </command_interface>
-          <state_interface name="position"/>
-          <state_interface name="velocity"/>
-        </joint>
-      </ros2_control>
-      <gazebo>
-        <plugin
-          filename="libgazebo_ros2_control.so"
-          name="gazebo_ros2_control">
-          <ros>
-            <remapping>~/cmd_vel_unstamped:=/cmd_vel</remapping>
-            <remapping>~/odom:=/odom</remapping>
-          </ros>
-          <parameters>$(find megarover_samples_ros2)/config/diff_drive_controller.yaml</parameters>
-        </plugin>
-      </gazebo>
-    </xacro:if>
-    <xacro:unless value="$(arg use_ros2_control)">
-      <!-- use libgazebo_ros_diff_drive.so -->
-      <gazebo>
-        <plugin
-          filename="libgazebo_ros_diff_drive.so"
-          name="diff_drive_controller">
-          <ros>
-            <namespace>/</namespace>
-          </ros>
-          <update_rate>50</update_rate>
-          <left_joint>left_wheel_joint</left_joint>
-          <right_joint>right_wheel_joint</right_joint>
-          <wheel_separation>0.284</wheel_separation>
-          <wheel_diameter>0.152</wheel_diameter>
-          <publish_odom>true</publish_odom>
-          <publish_odom_tf>true</publish_odom_tf>
-          <odometry_frame>odom</odometry_frame>
-          <robot_base_frame>base_footprint</robot_base_frame>
-        </plugin>
-      </gazebo>
-    </xacro:unless>
-  </xacro:if>
   <xacro:if value="${'$(arg gazebo)' == 'ignition'}">
     <xacro:if value="$(arg use_ros2_control)">

File: urdf/camera/camera.gazebo.xacro (robot description, xacro)
@@ -3,38 +3,4 @@
   <xacro:macro name="camera_gazebo_v0" params="gazebo prefix">
     <gazebo reference="${prefix}_camera_link">
-      <xacro:if value="${gazebo == 'classic'}">
-        <sensor name="${prefix}_camera_sensor" type="depth">
-          <pose>0 0 0 0 0 0</pose>
-          <update_rate>30.0</update_rate>
-          <camera name="camera">
-            <horizontal_fov>1.56207</horizontal_fov>
-            <image>
-              <width>640</width>
-              <height>400</height>
-              <format>R8G8B8</format>
-            </image>
-            <clip>
-              <near>0.02</near>
-              <far>8.0</far>
-            </clip>
-            <noise>
-              <type>gaussian</type>
-              <mean>0.0</mean>
-              <stddev>0.007</stddev>
-            </noise>
-          </camera>
-          <plugin name="camera_controller" filename="libgazebo_ros_camera.so">
-            <min_depth>0.2</min_depth>
-            <max_depth>8.0</max_depth>
-            <hack_baseline>0.07</hack_baseline>
-            <frame_name>camera_depth_link</frame_name>
-            <distortion_k1>0.0</distortion_k1>
-            <distortion_k2>0.0</distortion_k2>
-            <distortion_k3>0.0</distortion_k3>
-            <distortion_t1>0.0</distortion_t1>
-            <distortion_t2>0.0</distortion_t2>
-          </plugin>
-        </sensor>
-      </xacro:if>
       <xacro:if value="${gazebo == 'ignition'}">
         <sensor name="${prefix}_camera_sensor" type="rgbd_camera">

File: urdf/lrf/lrf.gazebo.xacro (robot description, xacro)
@@ -3,39 +3,4 @@
   <xacro:macro name="lrf_gazebo_v0" params="gazebo prefix min_rad max_rad min_range max_range">
     <gazebo reference="${prefix}_lrf_link">
-      <xacro:if value="${gazebo == 'classic'}">
-        <sensor type="ray" name="${prefix}_lrf_sensor">
-          <pose>0 0 0 0 0 0</pose>
-          <visualize>false</visualize>
-          <update_rate>40</update_rate>
-          <ray>
-            <scan>
-              <horizontal>
-                <samples>1000</samples>
-                <resolution>1</resolution>
-                <min_angle>${min_rad}</min_angle>
-                <max_angle>${max_rad}</max_angle>
-              </horizontal>
-            </scan>
-            <range>
-              <min>${min_range}</min>
-              <max>${max_range}</max>
-              <resolution>0.001</resolution>
-            </range>
-            <noise>
-              <type>gaussian</type>
-              <mean>0.0</mean>
-              <stddev>0.03</stddev>
-            </noise>
-          </ray>
-          <plugin name='gazebo_ros_${prefix}_lrf_controller' filename='libgazebo_ros_ray_sensor.so'>
-            <ros>
-              <remapping>~/out:=scan</remapping>
-            </ros>
-            <output_type>sensor_msgs/LaserScan</output_type>
-            <!-- <frame_name> ommited, will default to ${prefix}_lrf_link-->
-            <frame_name>${prefix}_lrf_link</frame_name>
-          </plugin>
-        </sensor>
-      </xacro:if>
       <xacro:if value="${gazebo == 'ignition'}">
         <sensor type="gpu_lidar" name="${prefix}_lrf_sensor">

Commit message: removed unused code

File: robots/vmegarover.urdf.xacro (robot description, xacro)
@@ -1,5 +1,4 @@
 <?xml version="1.0"?>
 <robot name="vmegarover" xmlns:xacro="http://ros.org/wiki/xacro">
-  <xacro:arg name="gazebo" default="ignition" />
   <xacro:arg name="use_ros2_control" default="false" />
   <xacro:include filename="$(find megarover_samples_ros2)/urdf/body/vbody.urdf.xacro"/>
@@ -58,89 +57,73 @@
     <child link="camera_depth_link"/>
   </joint>
-  <xacro:if value="${'$(arg gazebo)' == 'ignition'}">
-    <xacro:if value="$(arg use_ros2_control)">
-      <!-- use ros2_control -->
-      <ros2_control name="GazeboSystem" type="system">
-        <hardware>
-          <!-- Garden or later -->
-          <!--
-          <plugin>gz_ros2_control/GazeboSimSystem</plugin>
-          -->
-          <plugin>ign_ros2_control/IgnitionSystem</plugin>
-        </hardware>
-        <joint name="left_wheel_joint">
-          <command_interface name="velocity">
-            <param name="min">-1</param>
-            <param name="max">1</param>
-          </command_interface>
-          <state_interface name="position"/>
-          <state_interface name="velocity"/>
-        </joint>
-        <joint name="right_wheel_joint">
-          <command_interface name="velocity">
-            <param name="min">-1</param>
-            <param name="max">1</param>
-          </command_interface>
-          <state_interface name="position"/>
-          <state_interface name="velocity"/>
-        </joint>
-      </ros2_control>
-      <gazebo>
+  <xacro:if value="$(arg use_ros2_control)">
+    <!-- use ros2_control -->
+    <ros2_control name="GazeboSystem" type="system">
+      <hardware>
         <!-- Garden or later -->
-        <!--
-        <plugin
-          filename="gz_ros2_control-system"
-          name="gz_ros2_control::GazeboSimROS2ControlPlugin">
-        -->
-        <plugin
-          filename="ign_ros2_control-system"
-          name="ign_ros2_control::IgnitionROS2ControlPlugin">
-          <parameters>$(find megarover_samples_ros2)/config/diff_drive_controller.yaml</parameters>
-          <ros>
-            <remapping>~/cmd_vel_unstamped:=/cmd_vel</remapping>
-            <remapping>~/odom:=/odom</remapping>
-          </ros>
-        </plugin>
-      </gazebo>
-    </xacro:if>
-    <xacro:unless value="$(arg use_ros2_control)">
-      <!-- use ignition-gazebo-diff-drive-system -->
-      <gazebo>
-        <!-- Garden or later -->
-        <!--
-        <plugin
-          filename="gz-sim-diff-drive-system"
-          name="gz::sim::systems::DiffDrive">
-        -->
-        <!-- Fortress -->
-        <plugin
-          filename="ignition-gazebo-diff-drive-system"
-          name="ignition::gazebo::systems::DiffDrive">
-          <left_joint>left_wheel_joint</left_joint>
-          <right_joint>right_wheel_joint</right_joint>
-          <wheel_separation>0.284</wheel_separation>
-          <wheel_radius>${0.152/2.0}</wheel_radius>
-          <odom_publish_frequency>50</odom_publish_frequency>
-          <!-- Limits -->
-          <!-- <max_linear_acceleration> 1.0</max_linear_acceleration> -->
-          <!-- <min_linear_acceleration>-1.0</min_linear_acceleration> -->
-          <!-- <max_angular_acceleration> 1.0</max_angular_acceleration> -->
-          <!-- <min_angular_acceleration>-1.0</min_angular_acceleration> -->
-          <!-- Output -->
-          <frame_id>odom</frame_id>
-          <child_frame_id>base_footprint</child_frame_id>
-          <!-- Topics -->
-          <topic>/cmd_vel</topic>
-          <odom_topic>/odom</odom_topic>
-          <tf_topic>/tf</tf_topic>
-        </plugin>
-        <plugin
-          filename="ignition-gazebo-joint-state-publisher-system"
-          name="ignition::gazebo::systems::JointStatePublisher">
-            <topic>/joint_states</topic>
-        </plugin>
-      </gazebo>
-    </xacro:unless>
+        <plugin>gz_ros2_control/GazeboSimSystem</plugin>
+      </hardware>
+      <joint name="left_wheel_joint">
+        <command_interface name="velocity">
+          <param name="min">-1</param>
+          <param name="max">1</param>
+        </command_interface>
+        <state_interface name="position"/>
+        <state_interface name="velocity"/>
+      </joint>
+      <joint name="right_wheel_joint">
+        <command_interface name="velocity">
+          <param name="min">-1</param>
+          <param name="max">1</param>
+        </command_interface>
+        <state_interface name="position"/>
+        <state_interface name="velocity"/>
+      </joint>
+    </ros2_control>
+    <gazebo>
+      <!-- Garden or later -->
+      <plugin
+        filename="gz_ros2_control-system"
+        name="gz_ros2_control::GazeboSimROS2ControlPlugin">
+        <parameters>$(find megarover_samples_ros2)/config/diff_drive_controller.yaml</parameters>
+        <ros>
+          <remapping>~/cmd_vel_unstamped:=/cmd_vel</remapping>
+          <remapping>~/odom:=/odom</remapping>
+        </ros>
+      </plugin>
+    </gazebo>
   </xacro:if>
+  <xacro:unless value="$(arg use_ros2_control)">
+    <!-- use gz-sim-diff-drive-system -->
+    <gazebo>
+      <!-- Garden or later -->
+      <plugin
+        filename="gz-sim-diff-drive-system"
+        name="gz::sim::systems::DiffDrive">
+        <left_joint>left_wheel_joint</left_joint>
+        <right_joint>right_wheel_joint</right_joint>
+        <wheel_separation>0.284</wheel_separation>
+        <wheel_radius>${0.152/2.0}</wheel_radius>
+        <odom_publish_frequency>50</odom_publish_frequency>
+        <!-- Limits -->
+        <!-- <max_linear_acceleration> 1.0</max_linear_acceleration> -->
+        <!-- <min_linear_acceleration>-1.0</min_linear_acceleration> -->
+        <!-- <max_angular_acceleration> 1.0</max_angular_acceleration> -->
+        <!-- <min_angular_acceleration>-1.0</min_angular_acceleration> -->
+        <!-- Output -->
+        <frame_id>odom</frame_id>
+        <child_frame_id>base_footprint</child_frame_id>
+        <!-- Topics -->
+        <topic>/cmd_vel</topic>
+        <odom_topic>/odom</odom_topic>
+        <tf_topic>/tf</tf_topic>
+      </plugin>
+      <plugin
+        filename="gz-sim-joint-state-publisher-system"
+        name="gz::sim::systems::JointStatePublisher">
+          <topic>/joint_states</topic>
+      </plugin>
+    </gazebo>
+  </xacro:unless>
   <!-- Base -->
   <xacro:base_gazebo_v0/>
@@ -158,12 +141,10 @@
   <!-- Camera -->
   <xacro:camera_gazebo_v0 gazebo="$(arg gazebo)" prefix="front"/>
-  <xacro:if value="${'$(arg gazebo)' == 'ignition'}">
-    <gazebo>
-      <plugin
-        filename="ignition-gazebo-sensors-system"
-        name="ignition::gazebo::systems::Sensors">
-        <render_engine>ogre2</render_engine>
-      </plugin>
-    </gazebo>
-  </xacro:if>
+  <gazebo>
+    <plugin
+      filename="gz-sim-sensors-system"
+      name="gz::sim::systems::Sensors">
+      <render_engine>ogre2</render_engine>
+    </plugin>
+  </gazebo>
 </robot>

File: urdf/camera/camera.gazebo.xacro (robot description, xacro)
@@ -3,30 +3,28 @@
   <xacro:macro name="camera_gazebo_v0" params="gazebo prefix">
     <gazebo reference="${prefix}_camera_link">
-      <xacro:if value="${gazebo == 'ignition'}">
-        <sensor name="${prefix}_camera_sensor" type="rgbd_camera">
-          <pose>0 0 0 0 0 0</pose>
-          <topic>${prefix}_camera_sensor</topic>
-          <update_rate>30.0</update_rate>
-          <gz_frame_id>${prefix}_camera_link</gz_frame_id>
-          <camera>
-            <horizontal_fov>1.56207</horizontal_fov>
-            <image>
-              <width>640</width>
-              <height>400</height>
-              <format>R8G8B8</format>
-            </image>
-            <clip>
-              <near>0.02</near>
-              <far>8.0</far>
-            </clip>
-            <optical_frame_id>camera_depth_link</optical_frame_id>
-            <noise>
-              <type>gaussian</type>
-              <mean>0.0</mean>
-              <stddev>0.007</stddev>
-            </noise>
-          </camera>
-        </sensor>
-      </xacro:if>
+      <sensor name="${prefix}_camera_sensor" type="rgbd_camera">
+        <pose>0 0 0 0 0 0</pose>
+        <topic>${prefix}_camera_sensor</topic>
+        <update_rate>30.0</update_rate>
+        <gz_frame_id>${prefix}_camera_link</gz_frame_id>
+        <camera>
+          <horizontal_fov>1.56207</horizontal_fov>
+          <image>
+            <width>640</width>
+            <height>400</height>
+            <format>R8G8B8</format>
+          </image>
+          <clip>
+            <near>0.02</near>
+            <far>8.0</far>
+          </clip>
+          <optical_frame_id>camera_depth_link</optical_frame_id>
+          <noise>
+            <type>gaussian</type>
+            <mean>0.0</mean>
+            <stddev>0.007</stddev>
+          </noise>
+        </camera>
+      </sensor>
     </gazebo>
   </xacro:macro>

File: urdf/lrf/lrf.gazebo.xacro (robot description, xacro)
@@ -3,33 +3,31 @@
   <xacro:macro name="lrf_gazebo_v0" params="gazebo prefix min_rad max_rad min_range max_range">
     <gazebo reference="${prefix}_lrf_link">
-      <xacro:if value="${gazebo == 'ignition'}">
-        <sensor type="gpu_lidar" name="${prefix}_lrf_sensor">
-          <pose>0 0 0 0 0 0</pose>
-          <topic>scan</topic>
-          <visualize>false</visualize>
-          <update_rate>40</update_rate>
-          <gz_frame_id>${prefix}_lrf_link</gz_frame_id>
-          <lidar>
-            <scan>
-              <horizontal>
-                <samples>1000</samples>
-                <resolution>1</resolution>
-                <min_angle>${min_rad}</min_angle>
-                <max_angle>${max_rad}</max_angle>
-              </horizontal>
-            </scan>
-            <range>
-              <min>${min_range}</min>
-              <max>${max_range}</max>
-              <resolution>0.001</resolution>
-            </range>
-            <noise>
-              <type>gaussian</type>
-              <mean>0.0</mean>
-              <stddev>0.03</stddev>
-            </noise>
-          </lidar>
-        </sensor>
-      </xacro:if>
+      <sensor type="gpu_lidar" name="${prefix}_lrf_sensor">
+        <pose>0 0 0 0 0 0</pose>
+        <topic>scan</topic>
+        <visualize>false</visualize>
+        <update_rate>40</update_rate>
+        <gz_frame_id>${prefix}_lrf_link</gz_frame_id>
+        <lidar>
+          <scan>
+            <horizontal>
+              <samples>1000</samples>
+              <resolution>1</resolution>
+              <min_angle>${min_rad}</min_angle>
+              <max_angle>${max_rad}</max_angle>
+            </horizontal>
+          </scan>
+          <range>
+            <min>${min_range}</min>
+            <max>${max_range}</max>
+            <resolution>0.001</resolution>
+          </range>
+          <noise>
+            <type>gaussian</type>
+            <mean>0.0</mean>
+            <stddev>0.03</stddev>
+          </noise>
+        </lidar>
+      </sensor>
     </gazebo>
   </xacro:macro>

Commit message: Change wheel collition to narrow contact points

File: robots/vmegarover.urdf.xacro (robot description, xacro)
@@ -15,10 +15,10 @@
   <!-- Right Wheel -->
   <xacro:wheel_v0 prefix="right" parent="base_link">
-    <origin xyz="0 -0.14199 0.074742"/>
+    <origin xyz="0 -0.142 0.074742"/>
     <axis xyz="0 1 0"/>
   </xacro:wheel_v0>
   <!-- Left Wheel -->
   <xacro:wheel_v0 prefix="left" parent="base_link">
-    <origin xyz="0 0.14199 0.074742"  rpy="0 0 ${M_PI}" />
+    <origin xyz="0 0.142 0.074742" rpy="0 0 ${M_PI}" />
     <axis xyz="0 -1 0"/>
   </xacro:wheel_v0>

File: urdf/body/body.gazebo.xacro (robot description, xacro)
@@ -4,6 +4,8 @@
     <gazebo reference="base_link">
       <selfCollide>false</selfCollide>
-      <mu1 value="0.0" />
-      <mu2 value="0.0" />
+      <mu1>0.0</mu1>
+      <mu2>0.0</mu2>
+      <kp>1000000.0</kp>
+      <kd>100.0</kd>
     </gazebo>
   </xacro:macro>

File: urdf/wheel/vwheel.urdf.xacro (robot description, xacro)
@@ -4,5 +4,6 @@
   <xacro:include filename="$(find megarover_samples_ros2)/urdf/wheel/wheel.gazebo.xacro"/>
   <xacro:property name="wheel_radius" value="0.076"/>
-  <xacro:property name="wheel_length" value="0.03"/>
+  <xacro:property name="wheel_inertial_length" value="0.03"/>
+  <xacro:property name="wheel_collition_length" value="0.001"/>
   <xacro:property name="wheel_mass" value="0.823"/>
   <xacro:macro name="wheel_v0" params="prefix parent *joint_origin *joint_axis">
@@ -22,5 +23,5 @@
         <origin xyz="0 0 0" rpy="${-M_PI/2} 0 0"/>
         <geometry>
-          <cylinder radius="${wheel_radius}" length="${wheel_length}"/>
+          <cylinder radius="${wheel_radius}" length="${wheel_collition_length}"/>
         </geometry>
       </collision>
@@ -28,5 +29,5 @@
         <origin xyz="0 0 0" rpy="${-M_PI/2} 0 0"/>
         <xacro:cylinder_inertial mass="${wheel_mass}"
-          radius="${wheel_radius}" length="${wheel_length}"/>
+          radius="${wheel_radius}" length="${wheel_inertial_length}"/>
       </inertial>
     </link>

File: urdf/wheel/wheel.gazebo.xacro (robot description, xacro)
@@ -4,6 +4,8 @@
     <gazebo reference="${prefix}_wheel_link">
       <selfCollide>false</selfCollide>
-      <mu1 value="1.0" />
-      <mu2 value="1.0" />
+      <mu1>1.0</mu1>
+      <mu2>1.0</mu2>
+      <kp>1000000.0</kp>
+      <kd>100.0</kd>
     </gazebo>
   </xacro:macro>

Commit message: Fix wheel rpy settings and update to avoit using M_PI

File: robots/vmegarover.urdf.xacro (robot description, xacro)
@@ -15,11 +15,15 @@
   <!-- Right Wheel -->
   <xacro:wheel_v0 prefix="right" parent="base_link">
-    <origin xyz="0 -0.142 0.074742"/>
-    <axis xyz="0 1 0"/>
+    <!-- Using M_PI causes an error in odometry. -->
+    <!-- <origin xyz="0 -0.142 0.074742" rpy="-${M_PI/2} 0 0"/> -->
+    <origin xyz="0 -0.142 0.074742" rpy="-1.57 0 0"/>
+    <axis xyz="0 0 1"/>
   </xacro:wheel_v0>
   <!-- Left Wheel -->
   <xacro:wheel_v0 prefix="left" parent="base_link">
-    <origin xyz="0 0.142 0.074742" rpy="0 0 ${M_PI}" />
-    <axis xyz="0 -1 0"/>
+    <!-- Using M_PI causes an error in odometry. -->
+    <!-- <origin xyz="0 0.142 0.074742" rpy="-${M_PI/2} 0 0"/> -->
+    <origin xyz="0 0.142 0.074742" rpy="-1.57 0 0"/>
+    <axis xyz="0 0 1"/>
   </xacro:wheel_v0>
   <!-- Front LRF -->

File: urdf/wheel/vwheel.urdf.xacro (robot description, xacro)
@@ -15,4 +15,10 @@
     <link name="${prefix}_wheel_link">
       <visual>
+        <xacro:if value="${prefix=='right'}">
+          <origin xyz="0 0 0" rpy="${M_PI/2} 0 0"/>
+        </xacro:if>
+        <xacro:if value="${prefix=='right'}">
+          <origin xyz="0 0 0" rpy="${M_PI/2} 0 0"/>
+        </xacro:if>
         <geometry>
           <mesh filename="file://$(find megarover_samples_ros2)/models/vmegarover/meshes/dae/vmega_wheel.dae"/>
@@ -20,5 +26,4 @@
       </visual>
       <collision>
-        <origin xyz="0 0 0" rpy="${-M_PI/2} 0 0"/>
         <geometry>
           <cylinder radius="${wheel_radius}" length="${wheel_length}"/>
@@ -26,5 +31,4 @@
       </collision>
       <inertial>
-        <origin xyz="0 0 0" rpy="${-M_PI/2} 0 0"/>
         <xacro:cylinder_inertial mass="${wheel_mass}"
           radius="${wheel_radius}" length="${wheel_length}"/>
