Commit message: update robot link

File: robots/vmegarover.urdf.xacro (robot description, xacro)
@@ -39,26 +39,8 @@
     <origin xyz="-0.289 0 0.1015"  rpy="0 0 ${M_PI}" />
   </xacro:lrf_v0 -->
-  <link name="lrf_link"/>
-  <joint name="lrf_link_joint" type="fixed">
-    <parent link="base_footprint"/>
-    <child link="lrf_link"/>
-    <origin xyz="0.099 0 0.1015"/>
-  </joint>
+  <!-- Front Camera -->
   <xacro:camera_v0 prefix="front" parent="base_link">
     <origin xyz="0.099 0 0.2515"/>
   </xacro:camera_v0>
-  <!-- Front Camera -->
-  <link name="camera_link"/>
-  <joint name="camera_link_joint" type="fixed">
-    <parent link="base_footprint"/>
-    <child link="camera_link"/>
-    <origin xyz="0.099 0 0.3015"/>
-  </joint>
-  <link name="camera_depth_link"/>
-  <joint name="camera_depth_joint" type="fixed">
-    <origin xyz="0 0 0" rpy="-1.57 0 -1.57"/>
-    <parent link="camera_link"/>
-    <child link="camera_depth_link"/>
-  </joint>
   <xacro:if value="$(arg use_ros2_control)">
     <!-- use ros2_control -->

File: urdf/camera/camera.gazebo.xacro (robot description, xacro)
@@ -7,5 +7,4 @@
         <topic>${prefix}_camera_sensor</topic>
         <update_rate>30.0</update_rate>
-        <gz_frame_id>${prefix}_camera_link</gz_frame_id>
         <camera>
           <horizontal_fov>1.56207</horizontal_fov>
@@ -19,5 +18,5 @@
             <far>8.0</far>
           </clip>
-          <optical_frame_id>camera_depth_link</optical_frame_id>
+          <optical_frame_id>${prefix}_camera_link</optical_frame_id>
           <noise>
             <type>gaussian</type>

File: urdf/camera/camera.urdf.xacro (robot description, xacro)
@@ -27,4 +27,10 @@
       </inertial>
     </link>
+    <link name="${prefix}_camera_optical_link"/>
+    <joint name="${prefix}_camera_optical_joint" type="fixed">
+      <origin xyz="0 0 0" rpy="-1.57 0 -1.57"/>
+      <parent link="${prefix}_camera_link"/>
+      <child link="${prefix}_camera_optical_link"/>
+    </joint>
   </xacro:macro>
 </robot>

Commit message: removed unnecessary description from URDF

File: robots/vmegarover.urdf.xacro (robot description, xacro)
@@ -36,26 +36,9 @@
     <origin xyz="-0.289 0 0.1015"  rpy="0 0 ${M_PI}" />
   </xacro:lrf_v0 -->
-  <link name="lrf_link"/>
-  <joint name="lrf_link_joint" type="fixed">
-    <parent link="base_footprint"/>
-    <child link="lrf_link"/>
-    <origin xyz="0.099 0 0.1015"/>
-  </joint>
+  <!-- Camera -->
+  <!-- Front Camera -->
   <xacro:camera_v0 prefix="front" parent="base_link">
     <origin xyz="0.099 0 0.2515"/>
   </xacro:camera_v0>
-  <!-- Front Camera -->
-  <link name="camera_link"/>
-  <joint name="camera_link_joint" type="fixed">
-    <parent link="base_footprint"/>
-    <child link="camera_link"/>
-    <origin xyz="0.099 0 0.3015"/>
-  </joint>
-  <link name="camera_depth_link"/>
-  <joint name="camera_depth_joint" type="fixed">
-    <origin xyz="0 0 0" rpy="-1.57 0 -1.57"/>
-    <parent link="camera_link"/>
-    <child link="camera_depth_link"/>
-  </joint>
   <!-- =============== Gazebo =============== -->
   <xacro:if value="${'$(arg gazebo)' == 'classic'}">

Commit message: removed unnecessary description

File: robots/vmegarover.urdf.xacro (robot description, xacro)
@@ -36,26 +36,7 @@
     <origin xyz="-0.289 0 0.1015"  rpy="0 0 ${M_PI}" />
   </xacro:lrf_v0 -->
-  <link name="lrf_link"/>
-  <joint name="lrf_link_joint" type="fixed">
-    <parent link="base_footprint"/>
-    <child link="lrf_link"/>
-    <origin xyz="0.099 0 0.1015"/>
-  </joint>
   <xacro:camera_v0 prefix="front" parent="base_link">
     <origin xyz="0.099 0 0.2515"/>
   </xacro:camera_v0>
-  <!-- Front Camera -->
-  <link name="camera_link"/>
-  <joint name="camera_link_joint" type="fixed">
-    <parent link="base_footprint"/>
-    <child link="camera_link"/>
-    <origin xyz="0.099 0 0.3015"/>
-  </joint>
-  <link name="camera_depth_link"/>
-  <joint name="camera_depth_joint" type="fixed">
-    <origin xyz="0 0 0" rpy="-1.57 0 -1.57"/>
-    <parent link="camera_link"/>
-    <child link="camera_depth_link"/>
-  </joint>
   <!-- =============== Gazebo =============== -->
   <xacro:if value="${'$(arg gazebo)' == 'classic'}">

Commit message: removed unnecessary description

File: robots/vmegarover.urdf.xacro (robot description, xacro)
@@ -33,10 +33,4 @@
     <origin xyz="-0.289 0 0.1015"  rpy="0 0 ${M_PI}" />
   </xacro:lrf_v0 -->
-  <link name="lrf_link"/>
-  <joint name="lrf_link_joint" type="fixed">
-    <parent link="base_footprint"/>
-    <child link="lrf_link"/>
-    <origin xyz="0.099 0 0.1015"/>
-  </joint>
   <!-- ===============  Transmission =============== -->
   <xacro:wheel_trans_v0 prefix="right"/>

Commit message: fixed URDF

File: robots/vmegarover.urdf.xacro (robot description, xacro)
@@ -16,6 +16,6 @@
   <xacro:wheel_v0 prefix="right" parent="base_link">
     <!-- Using M_PI causes an error in odometry. -->
-    <!-- <origin xyz="0 -0.142 0.074742" rpy="-${M_PI/2} 0 0"/> -->
-    <origin xyz="0 -0.142 0.074742" rpy="-1.57 0 0"/>
+    <!-- <origin xyz="0 -0.142 0.076" rpy="-${M_PI/2} 0 0"/> -->
+    <origin xyz="0 -0.142 0.076" rpy="-1.57 0 0"/>
     <axis xyz="0 0 1"/>
   </xacro:wheel_v0>
@@ -23,6 +23,6 @@
   <xacro:wheel_v0 prefix="left" parent="base_link">
     <!-- Using M_PI causes an error in odometry. -->
-    <!-- <origin xyz="0 0.142 0.074742" rpy="-${M_PI/2} 0 0"/> -->
-    <origin xyz="0 0.142 0.074742" rpy="-1.57 0 0"/>
+    <!-- <origin xyz="0 0.142 0.076" rpy="-${M_PI/2} 0 0"/> -->
+    <origin xyz="0 0.142 0.076" rpy="-1.57 0 0"/>
     <axis xyz="0 0 1"/>
   </xacro:wheel_v0>
@@ -90,11 +90,15 @@
         <right_joint>right_wheel_joint</right_joint>
         <wheel_separation>0.284</wheel_separation>
-        <wheel_radius>${0.152/2.0}</wheel_radius>
+        <wheel_radius>0.076</wheel_radius>
         <odom_publish_frequency>50</odom_publish_frequency>
         <!-- Limits -->
-        <!-- <max_linear_acceleration> 1.0</max_linear_acceleration> -->
-        <!-- <min_linear_acceleration>-1.0</min_linear_acceleration> -->
-        <!-- <max_angular_acceleration> 1.0</max_angular_acceleration> -->
-        <!-- <min_angular_acceleration>-1.0</min_angular_acceleration> -->
+        <max_linear_velocity>1.4</max_linear_velocity>
+        <min_linear_velocity>-1.4</min_linear_velocity>
+        <max_angular_velocity>3.0</max_angular_velocity>
+        <min_angular_velocity>-3.0</min_angular_velocity>
+        <max_linear_acceleration>2.0</max_linear_acceleration>
+        <min_linear_acceleration>-2.0</min_linear_acceleration>
+        <max_angular_acceleration>3.0</max_angular_acceleration>
+        <min_angular_acceleration>-3.0</min_angular_acceleration>
         <!-- Output -->
         <frame_id>odom</frame_id>

Commit message: fixed URDF

File: robots/vmegarover.urdf.xacro (robot description, xacro)
@@ -16,10 +16,10 @@
   <!-- Right Wheel -->
   <xacro:wheel_v0 prefix="right" parent="base_link">
-    <origin xyz="0 -0.14199 0.074742"/>
+    <origin xyz="0 -0.142 0.076"/>
     <axis xyz="0 1 0"/>
   </xacro:wheel_v0>
   <!-- Left Wheel -->
   <xacro:wheel_v0 prefix="left" parent="base_link">
-    <origin xyz="0 0.14199 0.074742"  rpy="0 0 ${M_PI}" />
+    <origin xyz="0 0.142 0.076"  rpy="0 0 ${M_PI}" />
     <axis xyz="0 -1 0"/>
   </xacro:wheel_v0>
@@ -161,11 +161,15 @@
           <right_joint>right_wheel_joint</right_joint>
           <wheel_separation>0.284</wheel_separation>
-          <wheel_radius>${0.152/2.0}</wheel_radius>
+          <wheel_radius>0.076</wheel_radius>
           <odom_publish_frequency>50</odom_publish_frequency>
           <!-- Limits -->
-          <!-- <max_linear_acceleration> 1.0</max_linear_acceleration> -->
-          <!-- <min_linear_acceleration>-1.0</min_linear_acceleration> -->
-          <!-- <max_angular_acceleration> 1.0</max_angular_acceleration> -->
-          <!-- <min_angular_acceleration>-1.0</min_angular_acceleration> -->
+          <max_linear_velocity>1.4</max_linear_velocity>
+          <min_linear_velocity>-1.4</min_linear_velocity>
+          <max_angular_velocity>3.0</max_angular_velocity>
+          <min_angular_velocity>-3.0</min_angular_velocity>
+          <max_linear_acceleration>2.0</max_linear_acceleration>
+          <min_linear_acceleration>-2.0</min_linear_acceleration>
+          <max_angular_acceleration>3.0</max_angular_acceleration>
+          <min_angular_acceleration>-3.0</min_angular_acceleration>
           <!-- Output -->
           <frame_id>odom</frame_id>

Commit message: updated URDF

File: robots/vmegarover.urdf.xacro (robot description, xacro)
@@ -16,11 +16,15 @@
   <!-- Right Wheel -->
   <xacro:wheel_v0 prefix="right" parent="base_link">
-    <origin xyz="0 -0.142 0.076"/>
-    <axis xyz="0 1 0"/>
+    <!-- Using M_PI causes an error in odometry. -->
+    <!-- <origin xyz="0 -0.142 0.076" rpy="-${M_PI/2} 0 0"/> -->
+    <origin xyz="0 -0.142 0.076" rpy="-1.57 0 0"/>
+    <axis xyz="0 0 1"/>
   </xacro:wheel_v0>
   <!-- Left Wheel -->
   <xacro:wheel_v0 prefix="left" parent="base_link">
-    <origin xyz="0 0.142 0.076"  rpy="0 0 ${M_PI}" />
-    <axis xyz="0 -1 0"/>
+    <!-- Using M_PI causes an error in odometry. -->
+    <!-- <origin xyz="0 0.142 0.076" rpy="-${M_PI/2} 0 0"/> -->
+    <origin xyz="0 0.142 0.076" rpy="-1.57 0 0"/>
+    <axis xyz="0 0 1"/>
   </xacro:wheel_v0>
   <!-- Front LRF -->

Commit message: refactor launch and URDF

File: robots/vmegarover.urdf.xacro (robot description, xacro)
@@ -138,13 +138,11 @@
   <xacro:wheel_gazebo_v0 prefix="left"/>
   <!-- LRF -->
-  <xacro:lrf_gazebo_v0 gazebo="$(arg gazebo)"
-                       prefix="front"
+  <xacro:lrf_gazebo_v0 prefix="front"
                        min_rad="-3.14" max_rad="3.14"
                        min_range="0.06" max_range="10.0"/>
-  <!-- xacro:lrf_gazebo_v0 gazebo="$(arg gazebo)"
-                       prefix="rear"
+  <!-- xacro:lrf_gazebo_v0 prefix="rear"
                        min_rad="-1.57" max_rad="1.57"
                        min_range="0.06" max_range="10.0"/ -->
   <!-- Camera -->
-  <xacro:camera_gazebo_v0 gazebo="$(arg gazebo)" prefix="front"/>
+  <xacro:camera_gazebo_v0 prefix="front"/>
 </robot>

File: urdf/camera/camera.gazebo.xacro (robot description, xacro)
@@ -1,5 +1,5 @@
 <?xml version="1.0"?>
 <robot xmlns:xacro="http://ros.org/wiki/xacro">
-  <xacro:macro name="camera_gazebo_v0" params="gazebo prefix">
+  <xacro:macro name="camera_gazebo_v0" params="prefix">
     <gazebo reference="${prefix}_camera_link">
       <sensor name="${prefix}_camera_sensor" type="rgbd_camera">

File: urdf/lrf/lrf.gazebo.xacro (robot description, xacro)
@@ -1,5 +1,5 @@
 <?xml version="1.0"?>
 <robot xmlns:xacro="http://ros.org/wiki/xacro">
-  <xacro:macro name="lrf_gazebo_v0" params="gazebo prefix min_rad max_rad min_range max_range">
+  <xacro:macro name="lrf_gazebo_v0" params="prefix min_rad max_rad min_range max_range">
     <gazebo reference="${prefix}_lrf_link">
       <sensor type="gpu_lidar" name="${prefix}_lrf_sensor">
